File: mixer.kicad_sch (KiCad schematic)
At the start: 24 parts, among them J3 3.5mm TRS, T1 T50-43, T2 T50-43, T3 T50-43, T4 T50-43

Commit message: Rework RF amplifier design and add AF amplification
Parts:
- removed C18, C19: 100n, symbol Device:C
- removed C20, C21: 10u, symbol Device:C_Polarized
- removed J3: 3.5mm TRS, symbol Connector_Audio:AudioJack3
- removed R17, R18: 100, symbol Device:R
- removed R19, R20: 270, symbol Device:R
- renumbered R15 to R22, R16 to R23, R21 to R24
Connections:
- net I_AF renamed AF_I
- net Q_AF renamed AF_Q
